File: OpenBikeSensor_pcb_flippedPower_b.sch (KiCad schematic (older format))
At the start: 17 parts, among them J2 Conn_01x04_Female, J3 Conn_01x04_Male, J4 Conn_01x04_Male, J5 Conn_01x05_Male, J7 Conn_01x06_Male, J8 Conn_01x06_Male, J9 Conn_01x06_Male, U1 ESP32-DEVKIT-32C, U3 XUNPU-TF-115-C266620

Commit message: MT3608 finished LM2596 removed LM285 moved
Parts:
- C1: Aliexpress (none) -> 123; Conrad (none) -> 123; Reichelt (none) -> 123; ebay (none) -> 123
Changed lines of the file:
@@
 F 2 "Capacitors_THT:C_Rect_L4.0mm_W2.5mm_P2.50mm" H 1250 2300 50  0001 C CNN
 F 3 "~" H 1250 2300 50  0001 C CNN
+F 4 "123" H 1250 2300 50  0001 C CNN "Reichelt"
+F 5 "123" H 1250 2300 50  0001 C CNN "Aliexpress"
+F 6 "123" H 1250 2300 50  0001 C CNN "Conrad"
+F 7 "123" H 1250 2300 50  0001 C CNN "ebay"
 	1    1250 2300
 	1    0    0    -1

Commit message: Elkos for SD Card added spme silk fixed all parts locked in position
Parts:
- added C2, C3: 22u, Capacitors_THT:CP_Radial_D4.0mm_P1.50mm, symbol device:CP_Small
- C1: footprint Capacitors_THT:C_Rect_L4.0mm_W2.5mm_P2.50mm -> Capacitors_THT:C_Disc_D3.0mm_W1.6mm_P2.50mm
Connections:
- wire segments 102 -> 107
Changed lines of the file:
@@
 	3550 6850 3350 6850
 Wire Wire Line
-	4950 6250 4750 6250
+	4950 6250 4900 6250
 Wire Wire Line
 	4750 7150 4900 7150
@@
 F 0 "C1" H 1000 2350 50  0000 L CNN
 F 1 "100n" H 950 2250 50  0000 L CNN
-F 2 "Capacitors_THT:C_Rect_L4.0mm_W2.5mm_P2.50mm" H 1250 2300 50  0001 C CNN
+F 2 "Capacitors_THT:C_Disc_D3.0mm_W1.6mm_P2.50mm" H 1250 2300 50  0001 C CNN
 F 3 "~" H 1250 2300 50  0001 C CNN
 F 4 "123" H 1250 2300 50  0001 C CNN "Reichelt"
@@
 Wire Notes Line
 	5350 1800 7650 1800
+Wire Wire Line
+	4900 6300 4900 6250
+Connection ~ 4900 6250
+Wire Wire Line
+	4900 6250 4750 6250
+Wire Wire Line
+	4900 6500 4900 6550
+Connection ~ 4900 6550
+Wire Wire Line
+	4900 6500 5050 6500
+Wire Wire Line
+	5050 6300 4900 6300
+$Comp
+L device:CP_Small C2
+U 1 1 5EE2E44B
+P 5050 6400
+F 0 "C2" H 5138 6446 50  0000 L CNN
+F 1 "22u" H 5138 6355 50  0000 L CNN
+F 2 "Capacitors_THT:CP_Radial_D4.0mm_P1.50mm" H 5050 6400 50  0001 C CNN
+F 3 "~" H 5050 6400 50  0001 C CNN
+	1    5050 6400
+	1    0    0    -1
+$EndComp
+$Comp
+L device:CP_Small C3
+U 1 1 5EE2EDDD
+P 4900 6400
+F 0 "C3" H 4650 6450 50  0000 L CNN
+F 1 "22u" H 4650 6350 50  0000 L CNN
+F 2 "Capacitors_THT:CP_Radial_D4.0mm_P1.50mm" H 4900 6400 50  0001 C CNN
+F 3 "~" H 4900 6400 50  0001 C CNN
+	1    4900 6400
+	1    0    0    -1
+$EndComp
+Connection ~ 4900 6300
+Connection ~ 4900 6500
 $EndSCHEMATC

Commit message: Panic Pullups for I2C added (in 0805) Gerber for JLCPCB added
Parts:
- added R6, R7: 10k, Resistors_SMD:R_0805_HandSoldering, symbol device:R_Small
Connections:
- wire segments 107 -> 111
Changed lines of the file:
@@
 Connection ~ 4900 6300
 Connection ~ 4900 6500
+$Comp
+L device:R_Small R6
+U 1 1 5EDA6EB5
+P 9700 3050
+F 0 "R6" H 9759 3096 50  0000 L CNN
+F 1 "10k" H 9759 3005 50  0000 L CNN
+F 2 "Resistors_SMD:R_0805_HandSoldering" H 9700 3050 50  0001 C CNN
+F 3 "~" H 9700 3050 50  0001 C CNN
+	1    9700 3050
+	-1   0    0    1
+$EndComp
+$Comp
+L device:R_Small R7
+U 1 1 5EDA73A1
+P 10050 3050
+F 0 "R7" H 10109 3096 50  0000 L CNN
+F 1 "10k" H 10109 3005 50  0000 L CNN
+F 2 "Resistors_SMD:R_0805_HandSoldering" H 10050 3050 50  0001 C CNN
+F 3 "~" H 10050 3050 50  0001 C CNN
+	1    10050 3050
+	-1   0    0    1
+$EndComp
+$Comp
+L power:+3.3V #PWR01
+U 1 1 5EDA777F
+P 9700 2800
+F 0 "#PWR01" H 9700 2650 50  0001 C CNN
+F 1 "+3.3V" V 9700 3050 50  0000 C CNN
+F 2 "" H 9700 2800 50  0001 C CNN
+F 3 "" H 9700 2800 50  0001 C CNN
+	1    9700 2800
+	1    0    0    -1
+$EndComp
+$Comp
+L power:+3.3V #PWR02
+U 1 1 5EDA824B
+P 10050 2800
+F 0 "#PWR02" H 10050 2650 50  0001 C CNN
+F 1 "+3.3V" V 10050 3050 50  0000 C CNN
+F 2 "" H 10050 2800 50  0001 C CNN
+F 3 "" H 10050 2800 50  0001 C CNN
+	1    10050 2800
+	1    0    0    -1
+$EndComp
+Text GLabel 9700 3300 3    50   Input ~ 0
+SDA
+Text GLabel 10050 3300 3    50   Input ~ 0
+SCL
+Wire Wire Line
+	9700 3150 9700 3300
+Wire Wire Line
+	10050 3150 10050 3300
+Wire Wire Line
+	10050 2950 10050 2800
+Wire Wire Line
+	9700 2950 9700 2800
 $EndSCHEMATC

Commit message: Connector for Neo-6M updated Now compatible with both variants of connectors
Parts:
- J2: footprint Pin_Headers:Pin_Header_Angled_1x04_Pitch2.54mm -> Pin_Headers:Pin_Header_Angled_1x05_Pitch2.54mm; symbol conn:Conn_01x04_Female -> conn:Conn_01x05_Female
Connections:
- wire segments 111 -> 112
Changed lines of the file:
@@
 	4900 6550 4900 6950
 $Comp
-L conn:Conn_01x04_Female J2
+L conn:Conn_01x05_Female J2
 U 1 1 5ED25A92
 P 5800 1200
-F 0 "J2" H 5692 1485 50  0000 C CNN
-F 1 "Conn_01x04_Female" H 5692 1394 50  0000 C CNN
-F 2 "Pin_Headers:Pin_Header_Angled_1x04_Pitch2.54mm" H 5800 1200 50  0001 C CNN
+F 0 "J2" H 5750 850 50  0000 C CNN
+F 1 "Conn_01x04_Female" H 4650 850 50  0000 C CNN
+F 2 "Pin_Headers:Pin_Header_Angled_1x05_Pitch2.54mm" H 5800 1200 50  0001 C CNN
 F 3 "~" H 5800 1200 50  0001 C CNN
 	1    5800 1200
@@
 P 6200 1300
 F 0 "#PWR08" H 6200 1050 50  0001 C CNN
-F 1 "GND" H 6205 1127 50  0000 C CNN
+F 1 "GND" V 6200 950 50  0000 C CNN
 F 2 "" H 6200 1300 50  0001 C CNN
 F 3 "" H 6200 1300 50  0001 C CNN
 	1    6200 1300
-	1    0    0    -1
+	0    -1   -1   0
 $EndComp
 Wire Wire Line
@@
 Wire Wire Line
 	9700 2950 9700 2800
+$Comp
+L power:+3.3V #PWR0122
+U 1 1 5EDCBF76
+P 6200 1400
+F 0 "#PWR0122" H 6200 1250 50  0001 C CNN
+F 1 "+3.3V" V 6200 1750 50  0000 C CNN
+F 2 "" H 6200 1400 50  0001 C CNN
+F 3 "" H 6200 1400 50  0001 C CNN
+	1    6200 1400
+	0    1    1    0
+$EndComp
+Wire Wire Line
+	6200 1400 6000 1400
 $EndSCHEMATC

Commit message: Bom updated
Parts:
- C1: Aliexpress 123 -> --; Conrad 123 -> https://www.conrad.de/de/p/tancap-ct4-0805y104m500c1t-keram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; Reichelt 123 -> https://www.reichelt.de/vielschicht-keramikkondensator-100n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; Segor.de (none) -> https://www.segor.de/#Q=u10-R2.5-X7R&M=1; ebay 123 -> --
- C2, C3: Aliexpress (none) -> --; Conrad (none) -> https://www.conrad.de/de/p/teapo-kss226m016s1a5b07k-elektro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; Optional (none) -> x; Reichelt (none) -> https://www.reichelt.de/elko-radial-22-uf-10-v-1000-h-low-e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; Segor.de (none) -> https://www.segor.de/#Q=ELRA22u-16%252F4x7&M=1; ebay (none) -> --
- D1: Aliexpress (none) -> --; Bemerkung (none) -> reichelt und Conrad nur LM385; Conrad (none) -> https://www.conrad.de/de/p/on-semiconductor-lm385z-1-2g-pmi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; Reichelt (none) -> https://www.reichelt.de/spannungsreferenz-fest-1-2-v-to-92-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; Segor.de (none) -> https://www.segor.de/#Q=LM285BXZ-1.2%252FSonder&M=1; ebay (none) -> --
- J2: Bemerkung (none) -> Neo-6M Module (Connector via Conrad/reichelt/segor); Conrad (none) -> https://www.conrad.de/de/p/tru-components-stiftleiste-stand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; Reichelt (none) -> https://www.reichelt.de/36pol-stiftleiste-gewinkelt-rm-2-54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; Segor.de (none) -> https://www.segor.de/#Q=SL1x40-90G&M=1
- J3: Aliexpress (none) -> https://de.aliexpress.com/item/32218396409.html; Bemerkung (none) -> Ultraschall Connector 1 (Connector via Conrad/reichelt/sego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; Conrad (none) -> https://www.conrad.de/de/p/bkl-electronic-stiftleiste-stand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; Reichelt (none) -> https://www.reichelt.de/40pol-stiftleiste-gerade-rm-2-54-sl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; Segor.de (none) -> https://www.segor.de/#Q=SL1x40-180G%252F13%252C8&M=1
- J4: Aliexpress (none) -> https://de.aliexpress.com/item/32218396409.html; Bemerkung (none) -> Ultraschall Connector 2 (Connector via Conrad/reichelt/sego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; Conrad (none) -> https://www.conrad.de/de/p/bkl-electronic-stiftleiste-stand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; Reichelt (none) -> https://www.reichelt.de/40pol-stiftleiste-gerade-rm-2-54-sl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; Segor.de (none) -> https://www.segor.de/#Q=SL1x40-180G%252F13%252C8&M=1
- J5: Bemerkung (none) -> Button/Display Connector; Conrad (none) -> https://www.conrad.de/de/p/bkl-electronic-stiftleiste-stand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; Reichelt (none) -> https://www.reichelt.de/40pol-stiftleiste-gerade-rm-2-54-sl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; Segor.de (none) -> https://www.segor.de/#Q=SL1x40-180G%252F13%252C8&M=1
- J7: Aliexpress (none) -> https://de.aliexpress.com/item/32899722811.html; Bemerkung (none) -> Micro SD Adapter (Connector via Conrad/reichelt/segor); Conrad (none) -> https://www.conrad.de/de/p/tru-components-stiftleiste-stand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; Reichelt (none) -> https://www.reichelt.de/36pol-stiftleiste-gewinkelt-rm-2-54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; Segor.de (none) -> https://www.segor.de/#Q=SL1x40-90G&M=1; ebay (none) -> https://www.ebay.de/itm/Micro-SD-Karten-SD-Card-Modul-SPI-f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
- J8: Bemerkung (none) -> Zusatz Connector 1; Conrad (none) -> https://www.conrad.de/de/p/bkl-electronic-stiftleiste-stand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; Optional (none) -> x; Reichelt (none) -> https://www.reichelt.de/40pol-stiftleiste-gerade-rm-2-54-sl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; Segor.de (none) -> https://www.segor.de/#Q=SL1x40-180G%252F13%252C8&M=1
- J9: Bemerkung (none) -> Zusatz Connector 2; Conrad (none) -> https://www.conrad.de/de/p/bkl-electronic-stiftleiste-stand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; Optional (none) -> x; Reichelt (none) -> https://www.reichelt.de/40pol-stiftleiste-gerade-rm-2-54-sl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; Segor.de (none) -> https://www.segor.de/#Q=SL1x40-180G%252F13%252C8&M=1
- R1: Reichelt (none) -> https://www.reichelt.de/widerstand-kohleschicht-10-kohm-020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; Segor.de (none) -> https://www.segor.de/#Q=MF10k-1%2525&M=1
- R2: Reichelt (none) -> https://www.reichelt.de/widerstand-metallschicht-1-0-mohm-0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; Segor.de (none) -> https://www.segor.de/#Q=MF5M6-1%2525&M=1
- R3: Reichelt (none) -> 2x https://www.reichelt.de/widerstand-metallschicht-1-0-moh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; Segor.de (none) -> 2x https://www.segor.de/#Q=MF5M6-1%2525&M=1
- R4: Conrad (none) -> https://www.conrad.de/de/p/yageo-cfr-25jt-52-150k-kohleschi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; Optional (none) -> x; Reichelt (none) -> https://www.reichelt.de/widerstand-kohleschicht-150-kohm-02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; Segor.de (none) -> https://www.segor.de/#Q=MF150k-1%2525&M=1
- R5: Conrad (none) -> https://www.conrad.de/de/p/tru-components-tc-1206s4f1503t5e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; Reichelt (none) -> https://www.reichelt.de/smd-widerstand-1206-150-kohm-125-mw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; Segor.de (none) -> https://www.segor.de/#Q=150k-1206-1%2525&M=1
- R6, R7: Optional (none) -> x
- SOCKET1: Bemerkung (none) -> SMD SD Card Slot; Conrad (none) -> --; Optional (none) -> x; Other Source (none) -> https://lcsc.com/product-detail/Card-Sockets-Connectors_XUN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; Reichelt (none) -> ---; Segor.de (none) -> --; ebay (none) -> --
- U1: Aliexpress (none) -> https://de.aliexpress.com/item/32889969250.html --- https:/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; Conrad (none) -> 2x https://www.conrad.de/de/p/fischer-elektronik-buchsenlei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; Reichelt (none) -> 2x https://www.reichelt.de/buchsenleisten-2-54-mm-1x16-gera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; Segor.de (none) -> https://www.segor.de/#Q=FL1x20-180G(h%253D5%252C7mm)&M=1 un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; ebay (none) -> https://www.ebay.de/itm/10-pcs-SMD-Buchsenleiste-1x-16-poli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
- U3: Bemerkung (none) -> SMD Micro SD Card Slot; Conrad (none) -> --; Optional (none) -> x; Other Source (none) -> https://lcsc.com/product-detail/Card-Sockets-Connectors_XUN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; Reichelt (none) -> --; Segor.de (none) -> --; ebay (none) -> --
Other:
- note added: "Messteil Akkuspannung \n(nach Schutzschaltung)\nR3 kann als 2x 5M in Reihe \nausgelegt werden.\n\nNur Verhältnis wichtig. \nNicht genauer Wert.\nMöglichst hochohmig!"
- note removed: "Messteil Akkuspannung \n(nach Schutzschaltung)\nR3 kann als 2x 5M in Reihe \nausgelegt werden"

Commit message: Verpolschutz hinzugefügt
Parts:
- U1: footprint ESP32-DEVKITC-32D:MODULE_ESP32-DEVKITC-32C_SMD -> ESP32-DEVKITC-32D:MODULE_ESP32-DEVKITC-32C_SMDBACKUP; Aliexpress https://de.aliexpress.com/item/32889969250.html --- https://de.aliexpress.com/item/32959541446.html -> https://de.aliexpress.com/item/32889969250.html --- https://de.aliexpress.com/item/32959541446.html --- https://de.aliexpress.com/item/33040503442.html --- https://de.aliexpress.com/item/4001050278803.html
Changed lines of the file:
@@
 F 0 "U1" H 3150 1667 50  0000 C CNN
 F 1 "ESP32-DEVKIT-32C" H 3150 1576 50  0000 C CNN
-F 2 "ESP32-DEVKITC-32D:MODULE_ESP32-DEVKITC-32C_SMD" H 3100 1600 50  0001 C CNN
+F 2 "ESP32-DEVKITC-32D:MODULE_ESP32-DEVKITC-32C_SMDBACKUP" H 3100 1600 50  0001 C CNN
 F 3 "" H 3100 1600 50  0001 C CNN
 F 4 "2x https://www.conrad.de/de/p/fischer-elektronik-buchsenleiste-standard-anzahl-reihen-1-polzahl-je-reihe-20-bl-lp-5-smd-20-z-1-409080.html" H 3100 1600 50  0001 C CNN "Conrad"
-F 5 "https://de.aliexpress.com/item/32889969250.html --- https://de.aliexpress.com/item/32959541446.html" H 3100 1600 50  0001 C CNN "Aliexpress"
+F 5 "https://de.aliexpress.com/item/32889969250.html --- https://de.aliexpress.com/item/32959541446.html --- https://de.aliexpress.com/item/33040503442.html  --- https://de.aliexpress.com/item/4001050278803.html" H 3100 1600 50  0001 C CNN "Aliexpress"
 F 6 "2x  https://www.reichelt.de/buchsenleisten-2-54-mm-1x16-gerade-mpe-094-1-016-p119919.html   und Beinchen wechselseitig umbiegen. Nur im Notfall!" H 3100 1600 50  0001 C CNN "Reichelt"
 F 7 "https://www.segor.de/#Q=FL1x20-180G(h%253D5%252C7mm)&M=1   und Beinchen wechselseitig umbiegen. Nur im Notfall!" H 3100 1600 50  0001 C CNN "Segor.de"

Commit message: Backup Pins added (6 IOs Vcc GND)
Parts:
- added J10: Conn_02x03_Odd_Even, Pin_Headers:Pin_Header_Straight_2x03_Pitch2.54mm_SMD, symbol conn:Conn_02x03_Odd_Even
Connections:
- net labels added: IO12, IO13, RX, TX, VN, VP
- wire segments 112 -> 124
Changed lines of the file:
@@
 Text Notes 7850 750  0    118  ~ 0
 Connector optical sensors
-$Sheet
-S 7800 3950 2450 650
-U 5EDE387A
-F0 "PowerPart" 118
-F1 "OpenBikeSensor_PowerPart.sch" 118
-$EndSheet
 Wire Notes Line
 	5350 3500 5350 1800
@@
 Wire Wire Line
 	6200 1400 6000 1400
+Text GLabel 2250 3000 0    39   Input ~ 0
+IO12
+Text GLabel 2250 3100 0    39   Input ~ 0
+IO13
+Wire Wire Line
+	2250 3000 2350 3000
+Wire Wire Line
+	2350 3100 2250 3100
+Text GLabel 4100 2100 2    39   Input ~ 0
+RX
+Text GLabel 4100 2200 2    39   Input ~ 0
+TX
+Wire Wire Line
+	4100 2100 3950 2100
+Wire Wire Line
+	4100 2200 3950 2200
+Text GLabel 6800 4400 2    39   Input ~ 0
+RX
+Text GLabel 6800 4300 2    39   Input ~ 0
+TX
+Text GLabel 6000 4400 0    39   Input ~ 0
+IO12
+Text GLabel 6000 4300 0    39   Input ~ 0
+IO13
+Wire Wire Line
+	6650 4400 6800 4400
+Wire Wire Line
+	6800 4300 6650 4300
+Wire Wire Line
+	6150 4400 6000 4400
+Wire Wire Line
+	6000 4300 6150 4300
+$Sheet
+S 7800 3950 2450 650
+U 5EDE387A
+F0 "PowerPart" 118
+F1 "OpenBikeSensor_PowerPart.sch" 118
+$EndSheet
+$Comp
+L conn:Conn_02x03_Odd_Even J10
+U 1 1 5EE8147C
+P 6450 4300
+F 0 "J10" H 6500 4617 50  0000 C CNN
+F 1 "Conn_02x03_Odd_Even" H 6500 4526 50  0000 C CNN
+F 2 "Pin_Headers:Pin_Header_Straight_2x03_Pitch2.54mm_SMD" H 6450 4300 50  0001 C CNN
+F 3 "~" H 6450 4300 50  0001 C CNN
+	1    6450 4300
+	-1   0    0    -1
+$EndComp
+Text GLabel 2200 2100 0    39   Input ~ 0
+VN
+Text GLabel 2200 2000 0    39   Input ~ 0
+VP
+Wire Wire Line
+	2200 2000 2350 2000
+Wire Wire Line
+	2350 2100 2200 2100
+Text GLabel 6000 4200 0    39   Input ~ 0
+VN
+Wire Wire Line
+	6150 4200 6000 4200
+Wire Wire Line
+	6650 4200 6800 4200
+Text GLabel 6800 4200 2    39   Input ~ 0
+VP
 $EndSCHEMATC

Commit message: Update to 0.02.04
Parts:
- removed D1: LM285Z-1.2, TO_SOT_Packages_THT:TO-92_Inline_Narrow_Oval, symbol references:LM285Z-1.2
- removed R4: 150k, Resistors_THT:R_Axial_DIN0207_L6.3mm_D2.5mm_P2.54mm_Vertical, symbol device:R_Small
- removed R5: 150k, Resistors_SMD:R_1206_HandSoldering, symbol device:R_Small
- added Q1: BS170, Package_TO_SOT_THT:TO-92_Inline, symbol Transistor_FET:BS170
Connections:
- net labels added: GPS_GND, GPS_GND_CONT
- net labels removed: VoltRef
- wire segments 124 -> 120
Changed lines of the file:
@@
 	1    0    0    -1
-$EndComp
-$Comp
-L power:GND #PWR08
-U 1 1 5ED28615
-P 6200 1300
-F 0 "#PWR08" H 6200 1050 50  0001 C CNN
-F 1 "GND" V 6200 950 50  0000 C CNN
-F 2 "" H 6200 1300 50  0001 C CNN
-F 3 "" H 6200 1300 50  0001 C CNN
-	1    6200 1300
-	0    -1   -1   0
 $EndComp
 Wire Wire Line
@@
 	1450 2500 1450 2400
 $Comp
-L references:LM285Z-1.2 D1
-U 1 1 5EDDD286
-P 8550 5850
-F 0 "D1" V 8641 5762 50  0000 R CNN
-F 1 "LM285Z-1.2" V 8550 5762 50  0000 R CNN
-F 2 "TO_SOT_Packages_THT:TO-92_Inline_Narrow_Oval" H 8550 5650 50  0001 C CIN
-F 3 "http://www.onsemi.com/pub_link/Collateral/LM285-D.PDF" V 8459 5762 50  0000 R CNN
-F 4 "--" H 8550 5850 50  0001 C CNN "Aliexpress"
-F 5 "reichelt und Conrad nur LM385" H 8550 5850 50  0001 C CNN "Bemerkung"
-F 6 "https://www.reichelt.de/spannungsreferenz-fest-1-2-v-to-92-lm-385-z1-2-p10492.html" H 8550 5850 50  0001 C CNN "Reichelt"
-F 7 "https://www.segor.de/#Q=LM285BXZ-1.2%252FSonder&M=1" H 8550 5850 50  0001 C CNN "Segor.de"
-F 8 "--" H 8550 5850 50  0001 C CNN "ebay"
-F 9 "https://www.conrad.de/de/p/on-semiconductor-lm385z-1-2g-pmic-spannungsreferenz-shunt-fest-to-92-174300.html" H 8550 5850 50  0001 C CNN "Conrad"
-	1    8550 5850
-	0    -1   -1   0
-$EndComp
-$Comp
 L power:GND #PWR022
 U 1 1 5EDDFE5E
-P 8550 6100
-F 0 "#PWR022" H 8550 5850 50  0001 C CNN
-F 1 "GND" H 8555 5927 50  0000 C CNN
-F 2 "" H 8550 6100 50  0001 C CNN
-F 3 "" H 8550 6100 50  0001 C CNN
-	1    8550 6100
-	1    0    0    -1
-$EndComp
-$Comp
-L device:R_Small R4
-U 1 1 5EDE0C4A
-P 8550 5500
-F 0 "R4" H 8609 5546 50  0000 L CNN
-F 1 "150k" H 8609 5455 50  0000 L CNN
-F 2 "Resistors_THT:R_Axial_DIN0207_L6.3mm_D2.5mm_P2.54mm_Vertical" H 8550 5500 50  0001 C CNN
-F 3 "~" H 8550 5500 50  0001 C CNN
-F 4 "x" H 8550 5500 50  0001 C CNN "Optional"
-F 5 "https://www.segor.de/#Q=MF150k-1%2525&M=1" H 8550 5500 50  0001 C CNN "Segor.de"
-F 6 "https://www.reichelt.de/widerstand-kohleschicht-150-kohm-0207-250-mw-5-1-4w-150k-p1355.html" H 8550 5500 50  0001 C CNN "Reichelt"
-F 7 "https://www.conrad.de/de/p/yageo-cfr-25jt-52-150k-kohleschicht-widerstand-150-k-axial-bedrahtet-0207-0-25-w-5-1-1417642.html" H 8550 5500 50  0001 C CNN "Conrad"
-	1    8550 5500
-	1    0    0    -1
-$EndComp
-$Comp
-L power:+3.3V #PWR021
-U 1 1 5EDE123E
-P 8550 5350
-F 0 "#PWR021" H 8550 5200 50  0001 C CNN
-F 1 "+3.3V" H 8565 5523 50  0000 C CNN
-F 2 "" H 8550 5350 50  0001 C CNN
-F 3 "" H 8550 5350 50  0001 C CNN
-	1    8550 5350
-	1    0    0    -1
-$EndComp
-Wire Wire Line
-	8550 6100 8550 6000
-Wire Wire Line
-	8550 5700 8550 5650
-Wire Wire Line
-	8550 5350 8550 5400
-Text GLabel 8450 5650 0    50   Input ~ 0
-VoltRef
-Wire Wire Line
-	8450 5650 8550 5650
-Connection ~ 8550 5650
-Wire Wire Line
-	8550 5650 8550 5600
+P 8850 6150
+F 0 "#PWR022" H 8850 5900 50  0001 C CNN
+F 1 "GND" H 8855 5977 50  0000 C CNN
+F 2 "" H 8850 6150 50  0001 C CNN
+F 3 "" H 8850 6150 50  0001 C CNN
+	1    8850 6150
+	1    0    0    -1
+$EndComp
+Wire Wire Line
+	8850 6150 8850 6050
+Text GLabel 8450 5850 0    50   Input ~ 0
+GPS_GND_CONT
 Text GLabel 2200 2300 0    50   Input ~ 0
-VoltRef
+GPS_GND_CONT
 Wire Wire Line
 	2200 2300 2350 2300
-$Comp
-L device:R_Small R5
-U 1 1 5EDFEA4B
-P 9000 5500
-F 0 "R5" H 9059 5546 50  0000 L CNN
-F 1 "150k" H 9059 5455 50  0000 L CNN
-F 2 "Resistors_SMD:R_1206_HandSoldering" H 9000 5500 50  0001 C CNN
-F 3 "~" H 9000 5500 50  0001 C CNN
-F 4 "https://www.segor.de/#Q=150k-1206-1%2525&M=1" H 9000 5500 50  0001 C CNN "Segor.de"
-F 5 "https://www.reichelt.de/smd-widerstand-1206-150-kohm-125-mw-0-1-spr-1206-150k-p123462.html" H 9000 5500 50  0001 C CNN "Reichelt"
-F 6 "https://www.conrad.de/de/p/tru-components-tc-1206s4f1503t5e203-dickschicht-widerstand-150-k-smd-1206-0-25-w-1-1-1584522.html" H 9000 5500 50  0001 C CNN "Conrad"
-	1    9000 5500
-	1    0    0    -1
-$EndComp
-Wire Wire Line
-	9000 5600 8550 5600
-Connection ~ 8550 5600
-Wire Wire Line
-	8550 5400 9000 5400
-Connection ~ 8550 5400
 Wire Notes Line
 	7900 4850 11050 4850
@@
 Text GLabel 6800 4200 2    39   Input ~ 0
 VP
+$Comp
+L Transistor_FET:BS170 Q1
+U 1 1 5F24A00D
+P 8750 5850
+F 0 "Q1" H 8956 5896 50  0000 L CNN
+F 1 "BS170" H 8956 5805 50  0000 L CNN
+F 2 "Package_TO_SOT_THT:TO-92_Inline" H 8950 5775 50  0001 L CIN
+F 3 "http://www.fairchildsemi.com/ds/BS/BS170.pdf" H 8750 5850 50  0001 L CNN
+	1    8750 5850
+	1    0    0    -1
+$EndComp
+Wire Wire Line
+	8450 5850 8550 5850
+Text GLabel 8850 5600 1    59   Input ~ 0
+GPS_GND
+Wire Wire Line
+	8850 5600 8850 5650
+Text GLabel 6200 1300 2    59   Input ~ 0
+GPS_GND
 $EndSCHEMATC
