File: OpenBikeSensor_pcb_flippedPower_b.sch (KiCad schematic (older format))
At the start: 20 parts, among them J10 Conn_02x03_Odd_Even, J2 Conn_01x04_Female, J3 Conn_01x04_Male, J4 Conn_01x04_Male, J5 Conn_01x05_Male, J7 Conn_01x06_Male, J8 Conn_01x06_Male, J9 Conn_01x06_Male, Q1 BS170, U1 ESP32-DEVKIT-32C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

Commit message: Switched GPS transistor to IO12 Updatet schematic and gerbers update 00.02.08
Parts:
- R2: value 5M -> 150k
- R3: value 10M -> 300k
Connections:
- net labels added: IO35
- net labels removed: IO12
Changed lines of the file:
@@
 P 1450 2000
 F 0 "R2" H 1509 2046 50  0000 L CNN
-F 1 "5M" H 1509 1955 50  0000 L CNN
+F 1 "150k" H 1509 1955 50  0000 L CNN
 F 2 "Resistors_THT:R_Axial_DIN0207_L6.3mm_D2.5mm_P2.54mm_Vertical" H 1450 2000 50  0001 C CNN
 F 3 "~" H 1450 2000 50  0001 C CNN
@@
 P 1450 2300
 F 0 "R3" H 1509 2346 50  0000 L CNN
-F 1 "10M" H 1509 2255 50  0000 L CNN
+F 1 "300k" H 1509 2255 50  0000 L CNN
 F 2 "Resistors_THT:R_Axial_DIN0207_L6.3mm_D2.5mm_P2.54mm_Vertical" H 1450 2300 50  0001 C CNN
 F 3 "~" H 1450 2300 50  0001 C CNN
@@
 Text GLabel 8450 5850 0    50   Input ~ 0
 GPS_GND_CONT
-Text GLabel 2200 2300 0    50   Input ~ 0
+Text GLabel 2250 3000 0    50   Input ~ 0
 GPS_GND_CONT
-Wire Wire Line
-	2200 2300 2350 2300
 Wire Notes Line
 	7900 4850 11050 4850
@@
 Text Notes 750  1350 0    118  ~ 0
 ESP32 Board
-Text Notes 750  3600 0    59   ~ 0
+Text Notes 800  3950 0    59   ~ 0
 Messteil Akkuspannung \n(nach Schutzschaltung)\nR3 kann als 2x 5M in Reihe \nausgelegt werden.\n\nNur Verhältnis wichtig. \nNicht genauer Wert.\nMöglichst hochohmig!
-Text Notes 2050 3950 0    59   ~ 0
+Text Notes 2050 4250 0    59   ~ 0
 Unbedingt auf Pinbelegung des ESP32 Bords achten!\nDieses Board hat 30 Pins. Manche Boards haben \nauch 38 Pins. Diese sind sehr ähnlich, \naber NICHT pinkompatibel. GND Pins zwischen IOs!
 Text Notes 5400 2050 0    118  ~ 0
@@
 Wire Wire Line
 	6200 1400 6000 1400
-Text GLabel 2250 3000 0    39   Input ~ 0
-IO12
+Text GLabel 2200 2300 0    39   Input ~ 0
+IO35
 Text GLabel 2250 3100 0    39   Input ~ 0
 IO13
-Wire Wire Line
-	2250 3000 2350 3000
 Wire Wire Line
 	2350 3100 2250 3100
@@
 TX
 Text GLabel 6000 4400 0    39   Input ~ 0
-IO12
+IO35
 Text GLabel 6000 4300 0    39   Input ~ 0
 IO13
@@
 Text GLabel 6200 1300 2    59   Input ~ 0
 GPS_GND
+Wire Wire Line
+	2200 2300 2350 2300
+Wire Wire Line
+	2350 3000 2250 3000
 $EndSCHEMATC
