File: OpenBikeSensor_pcb_flippedPower_b.sch (KiCad schematic (older format))
At the start: 20 parts, among them J10 Conn_02x03_Odd_Even, J2 Conn_01x04_Female, J3 Conn_01x04_Male, J4 Conn_01x04_Male, J5 Conn_01x05_Male, J7 Conn_01x06_Male, J8 Conn_01x06_Male, J9 Conn_01x06_Male, Q1 BS170, U1 ESP32-DEVKIT-32C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

Commit message: Updated BOM_for_soldering_Rev_0.03.10.html "Bemerkungen" have to be updated!
Parts:
- R6, R7: value 10k -> 1k2; Optional x -> (none)
Changed lines of the file:
@@
 P 9700 3050
 F 0 "R6" H 9759 3096 50  0000 L CNN
-F 1 "10k" H 9759 3005 50  0000 L CNN
+F 1 "1k2" H 9759 3005 50  0000 L CNN
 F 2 "Resistors_SMD:R_0805_HandSoldering" H 9700 3050 50  0001 C CNN
 F 3 "~" H 9700 3050 50  0001 C CNN
-F 4 "x" H 9700 3050 50  0001 C CNN "Optional"
+F 4 "" H 9700 3050 50  0001 C CNN "Optional"
 	1    9700 3050
 	-1   0    0    1
@@
 P 10050 3050
 F 0 "R7" H 10109 3096 50  0000 L CNN
-F 1 "10k" H 10109 3005 50  0000 L CNN
+F 1 "1k2" H 10109 3005 50  0000 L CNN
 F 2 "Resistors_SMD:R_0805_HandSoldering" H 10050 3050 50  0001 C CNN
 F 3 "~" H 10050 3050 50  0001 C CNN
-F 4 "x" H 10050 3050 50  0001 C CNN "Optional"
+F 4 "" H 10050 3050 50  0001 C CNN "Optional"
 	1    10050 3050
 	-1   0    0    1

Commit message: clean up model references and add missing libraries
Parts:
- C1: symbol device:C_Small -> Device:C_Small
- C2, C3: symbol device:CP_Small -> Device:CP_Small
- J10: footprint Pin_Headers:Pin_Header_Straight_2x03_Pitch2.54mm_SMD -> Connector_PinHeader_2.54mm:PinHeader_2x03_P2.54mm_Vertical; symbol conn:Conn_02x03_Odd_Even -> Connector_Generic:Conn_02x03_Odd_Even
- J2: footprint Pin_Headers:Pin_Header_Angled_1x05_Pitch2.54mm -> Connector_PinHeader_2.54mm:PinHeader_1x05_P2.54mm_Horizontal; symbol conn:Conn_01x05_Female -> Connector:Conn_01x05_Female
- J3, J4: footprint Pin_Headers:Pin_Header_Straight_1x04_Pitch2.54mm -> Connector_PinHeader_2.54mm:PinHeader_1x04_P2.54mm_Vertical; symbol conn:Conn_01x04_Male -> Connector:Conn_01x04_Male
- J5: footprint Pin_Headers:Pin_Header_Straight_1x05_Pitch2.54mm -> Connector_PinHeader_2.54mm:PinHeader_1x05_P2.54mm_Vertical; symbol conn:Conn_01x05_Male -> Connector:Conn_01x05_Male
- J7: footprint Pin_Headers:Pin_Header_Straight_1x06_Pitch2.54mm -> Connector_PinHeader_2.54mm:PinHeader_1x05_P2.54mm_Vertical; symbol conn:Conn_01x06_Male -> Connector:Conn_01x05_Male
- J8, J9: footprint Pin_Headers:Pin_Header_Straight_1x06_Pitch2.54mm -> Connector_PinHeader_2.54mm:PinHeader_1x06_P2.54mm_Vertical
- R1, R2, R3: footprint Resistors_THT:R_Axial_DIN0207_L6.3mm_D2.5mm_P2.54mm_Vertical -> Resistor_THT:R_Axial_DIN0207_L6.3mm_D2.5mm_P2.54mm_Vertical; symbol device:R_Small -> Device:R_Small
- R6, R7: symbol device:R_Small -> Device:R_Small
Changed lines of the file:
@@
 EESchema Schematic File Version 4
-LIBS:OpenBikeSensor_pcb_flippedPower_b-cache
 EELAYER 30 0
 EELAYER END
@@
 	4900 6550 4900 6950
 $Comp
-L conn:Conn_01x05_Female J2
+L Connector:Conn_01x05_Female J2
 U 1 1 5ED25A92
 P 5800 1200
 F 0 "J2" H 5750 850 50  0000 C CNN
 F 1 "Conn_01x04_Female" H 4650 850 50  0000 C CNN
-F 2 "Pin_Headers:Pin_Header_Angled_1x05_Pitch2.54mm" H 5800 1200 50  0001 C CNN
+F 2 "Connector_PinHeader_2.54mm:PinHeader_1x05_P2.54mm_Horizontal" H 5800 1200 50  0001 C CNN
 F 3 "~" H 5800 1200 50  0001 C CNN
 F 4 "Neo-6M Module (Connector via Conrad/reichelt/segor)" H 5800 1200 50  0001 C CNN "Bemerkung"
@@
 	4150 3300 3950 3300
 $Comp
-L conn:Conn_01x04_Male J3
+L Connector:Conn_01x04_Male J3
 U 1 1 5ED6A6B4
 P 5850 2400
 F 0 "J3" H 5958 2681 50  0000 C CNN
 F 1 "Conn_01x04_Male" H 5958 2590 50  0000 C CNN
-F 2 "Pin_Headers:Pin_Header_Straight_1x04_Pitch2.54mm" H 5850 2400 50  0001 C CNN
+F 2 "Connector_PinHeader_2.54mm:PinHeader_1x04_P2.54mm_Vertical" H 5850 2400 50  0001 C CNN
 F 3 "~" H 5850 2400 50  0001 C CNN
 F 4 "Ultraschall Connector 1 (Connector via Conrad/reichelt/segor)" H 5850 2400 50  0001 C CNN "Bemerkung"
@@
 $EndComp
 $Comp
-L conn:Conn_01x04_Male J4
+L Connector:Conn_01x04_Male J4
 U 1 1 5ED6B21F
 P 5850 2950
 F 0 "J4" H 5958 3231 50  0000 C CNN
 F 1 "Conn_01x04_Male" H 5958 3140 50  0000 C CNN
-F 2 "Pin_Headers:Pin_Header_Straight_1x04_Pitch2.54mm" H 5850 2950 50  0001 C CNN
+F 2 "Connector_PinHeader_2.54mm:PinHeader_1x04_P2.54mm_Vertical" H 5850 2950 50  0001 C CNN
 F 3 "~" H 5850 2950 50  0001 C CNN
 F 4 "Ultraschall Connector 2 (Connector via Conrad/reichelt/segor)" H 5850 2950 50  0001 C CNN "Bemerkung"
@@
 	3950 3100 4150 3100
 $Comp
-L conn:Conn_01x05_Male J5
+L Connector:Conn_01x05_Male J5
 U 1 1 5ED82C02
 P 8200 3050
 F 0 "J5" H 8308 3431 50  0000 C CNN
 F 1 "Conn_01x05_Male" H 8308 3340 50  0000 C CNN
-F 2 "Pin_Headers:Pin_Header_Straight_1x05_Pitch2.54mm" H 8200 3050 50  0001 C CNN
+F 2 "Connector_PinHeader_2.54mm:PinHeader_1x05_P2.54mm_Vertical" H 8200 3050 50  0001 C CNN
 F 3 "~" H 8200 3050 50  0001 C CNN
 F 4 "Button/Display Connector" H 8200 3050 50  0001 C CNN "Bemerkung"
@@
 	8600 2850 8400 2850
 $Comp
-L conn:Conn_01x06_Male J7
+L Connector:Conn_01x05_Male J7
 U 1 1 5EDB38F7
 P 5650 5950
 F 0 "J7" H 5758 6331 50  0000 C CNN
 F 1 "Conn_01x06_Male" H 5758 6240 50  0000 C CNN
-F 2 "Pin_Headers:Pin_Header_Straight_1x06_Pitch2.54mm" H 5650 5950 50  0001 C CNN
+F 2 "Connector_PinHeader_2.54mm:PinHeader_1x05_P2.54mm_Vertical" H 5650 5950 50  0001 C CNN
 F 3 "~" H 5650 5950 50  0001 C CNN
 F 4 "https://de.aliexpress.com/item/32899722811.html" H 5650 5950 50  0001 C CNN "Aliexpress"
@@
 	5850 6250 6000 6250
 $Comp
-L device:R_Small R1
+L Device:R_Small R1
 U 1 1 5ED1D73B
 P 9250 3050
 F 0 "R1" H 9309 3096 50  0000 L CNN
 F 1 "10k" H 9309 3005 50  0000 L CNN
-F 2 "Resistors_THT:R_Axial_DIN0207_L6.3mm_D2.5mm_P2.54mm_Vertical" H 9250 3050 50  0001 C CNN
+F 2 "Resistor_THT:R_Axial_DIN0207_L6.3mm_D2.5mm_P2.54mm_Vertical" H 9250 3050 50  0001 C CNN
 F 3 "~" H 9250 3050 50  0001 C CNN
 F 4 "https://www.segor.de/#Q=MF10k-1%2525&M=1" H 9250 3050 50  0001 C CNN "Segor.de"
@@
 $EndComp
 $Comp
-L device:R_Small R2
+L Device:R_Small R2
 U 1 1 5ED66556
 P 1450 2000
 F 0 "R2" H 1509 2046 50  0000 L CNN
 F 1 "150k" H 1509 1955 50  0000 L CNN
-F 2 "Resistors_THT:R_Axial_DIN0207_L6.3mm_D2.5mm_P2.54mm_Vertical" H 1450 2000 50  0001 C CNN
+F 2 "Resistor_THT:R_Axial_DIN0207_L6.3mm_D2.5mm_P2.54mm_Vertical" H 1450 2000 50  0001 C CNN
 F 3 "~" H 1450 2000 50  0001 C CNN
 F 4 "https://www.segor.de/#Q=MF5M6-1%2525&M=1" H 1450 2000 50  0001 C CNN "Segor.de"
@@
 $EndComp
 $Comp
-L device:R_Small R3
+L Device:R_Small R3
 U 1 1 5ED66E45
 P 1450 2300
 F 0 "R3" H 1509 2346 50  0000 L CNN
 F 1 "300k" H 1509 2255 50  0000 L CNN
-F 2 "Resistors_THT:R_Axial_DIN0207_L6.3mm_D2.5mm_P2.54mm_Vertical" H 1450 2300 50  0001 C CNN
+F 2 "Resistor_THT:R_Axial_DIN0207_L6.3mm_D2.5mm_P2.54mm_Vertical" H 1450 2300 50  0001 C CNN
 F 3 "~" H 1450 2300 50  0001 C CNN
 F 4 "2x https://www.segor.de/#Q=MF5M6-1%2525&M=1" H 1450 2300 50  0001 C CNN "Segor.de"
@@
 	1450 2150 1450 2100
 $Comp
-L device:C_Small C1
+L Device:C_Small C1
 U 1 1 5ED7CAE9
 P 1250 2300
@@
 F 0 "J8" H 8108 1931 50  0000 C CNN
 F 1 "Conn_01x06_Male" H 8108 1840 50  0000 C CNN
-F 2 "Pin_Headers:Pin_Header_Straight_1x06_Pitch2.54mm" H 8000 1550 50  0001 C CNN
+F 2 "Connector_PinHeader_2.54mm:PinHeader_1x06_P2.54mm_Vertical" H 8000 1550 50  0001 C CNN
 F 3 "~" H 8000 1550 50  0001 C CNN
 F 4 "x" H 8000 1550 50  0001 C CNN "Optional"
@@
 F 0 "J9" H 10008 1931 50  0000 C CNN
 F 1 "Conn_01x06_Male" H 10008 1840 50  0000 C CNN
-F 2 "Pin_Headers:Pin_Header_Straight_1x06_Pitch2.54mm" H 9900 1550 50  0001 C CNN
+F 2 "Connector_PinHeader_2.54mm:PinHeader_1x06_P2.54mm_Vertical" H 9900 1550 50  0001 C CNN
 F 3 "~" H 9900 1550 50  0001 C CNN
 F 4 "x" H 9900 1550 50  0001 C CNN "Optional"
@@
 	5050 6300 4900 6300
 $Comp
-L device:CP_Small C2
+L Device:CP_Small C2
 U 1 1 5EE2E44B
 P 5050 6400
@@
 $EndComp
 $Comp
-L device:CP_Small C3
+L Device:CP_Small C3
 U 1 1 5EE2EDDD
 P 4900 6400
@@
 	1    0    0    -1
 $EndComp
-Connection ~ 4900 6300
-Connection ~ 4900 6500
-$Comp
-L device:R_Small R6
+$Comp
+L Device:R_Small R6
 U 1 1 5EDA6EB5
 P 9700 3050
@@
 $EndComp
 $Comp
-L device:R_Small R7
+L Device:R_Small R7
 U 1 1 5EDA73A1
 P 10050 3050
@@
 $EndSheet
 $Comp
-L conn:Conn_02x03_Odd_Even J10
+L Connector_Generic:Conn_02x03_Odd_Even J10
 U 1 1 5EE8147C
 P 6450 4300
 F 0 "J10" H 6500 4617 50  0000 C CNN
 F 1 "Conn_02x03_Odd_Even" H 6500 4526 50  0000 C CNN
-F 2 "Pin_Headers:Pin_Header_Straight_2x03_Pitch2.54mm_SMD" H 6450 4300 50  0001 C CNN
+F 2 "Connector_PinHeader_2.54mm:PinHeader_2x03_P2.54mm_Vertical" H 6450 4300 50  0001 C CNN
 F 3 "~" H 6450 4300 50  0001 C CNN
 	1    6450 4300
