File: OpenBikeSensor_pcb_flippedPower.sch (KiCad schematic (older format))
At the start: 19 parts, among them J1 Conn_01x02_Male, J2 Conn_01x04_Female, J3 Conn_01x04_Male, J4 Conn_01x04_Male, J5 Conn_01x05_Male, J6 Conn_01x02_Male, J7 Conn_01x06_Male, M1 LIPoChargerwithProtection, U1 ESP32-DEVKIT-32C, U2 LM2596_mini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

Commit message: wip
Parts:
- C1: symbol device:C_Small -> Device:C_Small
- D1: symbol references:LM285Z-1.2 -> Reference_Voltage:LM285Z-1.2
- J1, J6: symbol conn:Conn_01x02_Male -> Connector:Conn_01x02_Male
- J2: symbol conn:Conn_01x04_Female -> Connector:Conn_01x04_Female
- J3, J4: symbol conn:Conn_01x04_Male -> Connector:Conn_01x04_Male
- J5: symbol conn:Conn_01x05_Male -> Connector:Conn_01x05_Male
- J7: symbol conn:Conn_01x06_Male -> Connector:Conn_01x06_Male
- R1, R2, R3, R4, R5: symbol device:R_Small -> Device:R_Small
Changed lines of the file:
@@
 EESchema Schematic File Version 4
-LIBS:OpenBikeSensor_pcb-cache
 EELAYER 30 0
 EELAYER END
@@
 	4750 6550 4900 6550
 $Comp
-L conn:Conn_01x02_Male J1
+L Connector:Conn_01x02_Male J1
 U 1 1 5ED16B37
 P 5650 2800
@@
 	4900 6550 4900 6950
 $Comp
-L conn:Conn_01x04_Female J2
+L Connector:Conn_01x04_Female J2
 U 1 1 5ED25A92
 P 5750 1650
@@
 	9550 2850 9700 2850
 $Comp
-L conn:Conn_01x04_Male J3
+L Connector:Conn_01x04_Male J3
 U 1 1 5ED6A6B4
 P 5850 3700
@@
 $EndComp
 $Comp
-L conn:Conn_01x04_Male J4
+L Connector:Conn_01x04_Male J4
 U 1 1 5ED6B21F
 P 5850 4250
@@
 	3950 3100 4150 3100
 $Comp
-L conn:Conn_01x05_Male J5
+L Connector:Conn_01x05_Male J5
 U 1 1 5ED82C02
 P 8400 4100
@@
 	8800 3900 8600 3900
 $Comp
-L conn:Conn_01x02_Male J6
+L Connector:Conn_01x02_Male J6
 U 1 1 5ED902CA
 P 9950 2250
@@
 $EndComp
 $Comp
-L conn:Conn_01x06_Male J7
+L Connector:Conn_01x06_Male J7
 U 1 1 5EDB38F7
 P 5650 5950
@@
 $EndComp
 $Comp
-L device:R_Small R1
+L Device:R_Small R1
 U 1 1 5ED1D73B
 P 9450 4100
@@
 	9950 2450 10450 2450
 $Comp
-L device:R_Small R2
+L Device:R_Small R2
 U 1 1 5ED66556
 P 1450 2000
@@
 $EndComp
 $Comp
-L device:R_Small R3
+L Device:R_Small R3
 U 1 1 5ED66E45
 P 1450 2300
@@
 	1450 2150 1450 2100
 $Comp
-L device:C_Small C1
+L Device:C_Small C1
 U 1 1 5ED7CAE9
 P 1250 2300
@@
 	1450 2500 1450 2400
 $Comp
-L references:LM285Z-1.2 D1
+L Reference_Voltage:LM285Z-1.2 D1
 U 1 1 5EDDD286
 P 8550 5850
@@
 $EndComp
 $Comp
-L device:R_Small R4
+L Device:R_Small R4
 U 1 1 5EDE0C4A
 P 8550 5500
@@
 	2200 2300 2350 2300
 $Comp
-L device:R_Small R5
+L Device:R_Small R5
 U 1 1 5EDFEA4B
 P 9000 5500
@@
 Wire Wire Line
 	9000 5600 8550 5600
-Connection ~ 8550 5600
 Wire Wire Line
 	8550 5400 9000 5400
-Connection ~ 8550 5400
 Wire Notes Line
 	7900 4850 11050 4850
