File: OpenBikeSensor_PowerPart.sch (KiCad schematic (older format))
At the start: 5 parts, among them J1 Conn_01x02_Male, J6 Conn_01x02_Male, M1 LIPoChargerwithProtection, U2 LM2596_mini, U4 DCDC_fix

Commit message: MT3608 finished LM2596 removed LM285 moved
Parts:
- U2: footprint Custom_Modules:LM2596_Mini -> (none)
Changed lines of the file:
@@
 F 0 "U2" H 8525 2765 50  0000 C CNN
 F 1 "LM2596_mini" H 8525 2674 50  0000 C CNN
-F 2 "Custom_Modules:LM2596_Mini" H 8500 2650 50  0001 C CNN
+F 2 "" H 8500 2650 50  0001 C CNN
 F 3 "" H 8500 2650 50  0001 C CNN
 	1    8550 2300

Commit message: Bom updated
Parts:
- J1: Bemerkung (none) -> Batterie Connector (bevorzugt Reichelt da direkt als Kabels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; Conrad (none) -> https://www.conrad.de/de/p/bkl-electronic-stiftleiste-stand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; Reichelt (none) -> https://www.reichelt.de/platinensteckverbinder-gerade-weiss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; Segor.de (none) -> https://www.segor.de/#Q=SL1x40-180G%252F13%252C8&M=1
- J6: Bemerkung (none) -> Switch Connector; Conrad (none) -> https://www.conrad.de/de/p/bkl-electronic-stiftleiste-stand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; Reichelt (none) -> https://www.reichelt.de/40pol-stiftleiste-gerade-rm-2-54-sl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; Segor.de (none) -> https://www.segor.de/#Q=SL1x40-180G%252F13%252C8&M=1
- M1: Aliexpress (none) -> https://de.aliexpress.com/item/4000845174924.html; Conrad (none) -> --; Reichelt (none) -> --; Segor.de (none) -> --; ebay (none) -> https://www.ebay.de/itm/TP4056-USB-C-Neu-Li-Ion-Lademodul-5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
- U2: Optional (none) -> obsolet
- U4: Aliexpress (none) -> https://de.aliexpress.com/item/33029072332.html?spm=a2g0s.9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; ebay (none) -> https://www.ebay.de/itm/Automatic-Buck-Boost-Step-Up-Down-M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
Changed lines of the file:
@@
 F 2 "Custom_Modules:MT3608_SEPIC_DCDC" H 1650 1950 50  0001 C CNN
 F 3 "" H 1650 1950 50  0001 C CNN
+F 4 "https://de.aliexpress.com/item/33029072332.html?spm=a2g0s.9042311.0.0.3da24c4dCy9veI" H 1700 1600 50  0001 C CNN "Aliexpress"
+F 5 "https://www.ebay.de/itm/Automatic-Buck-Boost-Step-Up-Down-Module-DC-DC-2-5V-15V-To-3-3V-4-2V-5V-9V-12V/264075497616?_trksid=p2485497.m4902.l9144 " H 1700 1600 50  0001 C CNN "ebay"
 	1    1700 1600
 	1    0    0    -1
@@
 F 2 "" H 8500 2650 50  0001 C CNN
 F 3 "" H 8500 2650 50  0001 C CNN
+F 4 "obsolet" H 8550 2300 50  0001 C CNN "Optional"
 	1    8550 2300
 	1    0    0    -1
@@
 F 2 "Custom_Modules:BATTERY-CHARGER-LI-PROT" H 1550 3100 50  0001 C CNN
 F 3 "" H 1550 3100 50  0001 C CNN
+F 4 "https://de.aliexpress.com/item/4000845174924.html" H 1550 3100 50  0001 C CNN "Aliexpress"
+F 5 "https://www.ebay.de/itm/TP4056-USB-C-Neu-Li-Ion-Lademodul-5V-1A-18650-Laderegler-Charger-LIPO-Board/392521487361?hash=item5b641a9401:m:mVnUrPFcSEHHaEuYbWKFGEQ" H 1550 3100 50  0001 C CNN "ebay"
+F 6 "--" H 1550 3100 50  0001 C CNN "Conrad"
+F 7 "--" H 1550 3100 50  0001 C CNN "Reichelt"
+F 8 "--" H 1550 3100 50  0001 C CNN "Segor.de"
 	1    1550 3100
 	1    0    0    -1
@@
 F 2 "Pin_Headers:Pin_Header_Straight_1x02_Pitch2.54mm" H 2650 3100 50  0001 C CNN
 F 3 "~" H 2650 3100 50  0001 C CNN
+F 4 "Switch Connector" H 2650 3100 50  0001 C CNN "Bemerkung"
+F 5 "https://www.segor.de/#Q=SL1x40-180G%252F13%252C8&M=1" H 2650 3100 50  0001 C CNN "Segor.de"
+F 6 "https://www.reichelt.de/40pol-stiftleiste-gerade-rm-2-54-sl-1x40g-2-54-p19506.html" H 2650 3100 50  0001 C CNN "Reichelt"
+F 7 "https://www.conrad.de/de/p/bkl-electronic-stiftleiste-standard-anzahl-reihen-1-polzahl-je-reihe-40-10120513-1-393494.html" H 2650 3100 50  0001 C CNN "Conrad"
 	1    2650 3100
 	0    1    1    0
@@
 F 2 "Pin_Headers:Pin_Header_Straight_1x02_Pitch2.54mm" H 950 4450 50  0001 C CNN
 F 3 "~" H 950 4450 50  0001 C CNN
+F 4 "Batterie Connector (bevorzugt Reichelt da direkt als Kabelset!)" H 950 4450 50  0001 C CNN "Bemerkung"
+F 5 "https://www.conrad.de/de/p/bkl-electronic-stiftleiste-standard-anzahl-reihen-1-polzahl-je-reihe-40-10120513-1-393494.html" H 950 4450 50  0001 C CNN "Conrad"
+F 6 "https://www.reichelt.de/platinensteckverbinder-gerade-weiss-2-polig-ps-25-2g-ws-p14825.html" H 950 4450 50  0001 C CNN "Reichelt"
+F 7 "https://www.segor.de/#Q=SL1x40-180G%252F13%252C8&M=1" H 950 4450 50  0001 C CNN "Segor.de"
 	1    950  4450
 	1    0    0    -1

Commit message: Verpolschutz hinzugefügt
Parts:
- added D2: 1N4004, Diodes_THT:D_DO-41_SOD81_P10.16mm_Horizontal, symbol diode:1N4004
- added F1: Polyfuse, Fuse_Holders_and_Fuses:Fuse_TE5_Littlefuse-395Series, symbol device:Polyfuse
Connections:
- wire segments 19 -> 22
Other:
- note added: "Verpolschutz Battery"
Changed lines of the file:
@@
 Text Notes 750  4150 0    118  ~ 0
 Connector Battery
-Wire Wire Line
-	1150 4450 1550 4450
 $Comp
 L power:-BATT #PWR?
 U 1 1 5EE082A0
-P 1550 4550
+P 1050 6050
 AR Path="/5EE082A0" Ref="#PWR?"  Part="1"
 AR Path="/5EDE387A/5EE082A0" Ref="#PWR0120"  Part="1"
-F 0 "#PWR0120" H 1550 4400 50  0001 C CNN
-F 1 "-BATT" V 1565 4678 50  0000 L CNN
-F 2 "" H 1550 4550 50  0001 C CNN
-F 3 "" H 1550 4550 50  0001 C CNN
-	1    1550 4550
-	0    1    1    0
+F 0 "#PWR0120" H 1050 5900 50  0001 C CNN
+F 1 "-BATT" H 700 6100 50  0000 L CNN
+F 2 "" H 1050 6050 50  0001 C CNN
+F 3 "" H 1050 6050 50  0001 C CNN
+	1    1050 6050
+	-1   0    0    1
 $EndComp
 Wire Wire Line
@@
 L power:+BATT #PWR?
 U 1 1 5EE082A7
-P 1550 4450
+P 1050 5450
 AR Path="/5EE082A7" Ref="#PWR?"  Part="1"
 AR Path="/5EDE387A/5EE082A7" Ref="#PWR0121"  Part="1"
-F 0 "#PWR0121" H 1550 4300 50  0001 C CNN
-F 1 "+BATT" H 1565 4623 50  0000 C CNN
-F 2 "" H 1550 4450 50  0001 C CNN
-F 3 "" H 1550 4450 50  0001 C CNN
-	1    1550 4450
+F 0 "#PWR0121" H 1050 5300 50  0001 C CNN
+F 1 "+BATT" H 1065 5623 50  0000 C CNN
+F 2 "" H 1050 5450 50  0001 C CNN
+F 3 "" H 1050 5450 50  0001 C CNN
+	1    1050 5450
 	1    0    0    -1
 $EndComp
@@
 	1    0    0    -1
 $EndComp
+$Comp
+L device:Polyfuse F1
+U 1 1 5EE15FB8
+P 1750 4450
+F 0 "F1" V 1525 4450 50  0000 C CNN
+F 1 "Polyfuse" V 1616 4450 50  0000 C CNN
+F 2 "Fuse_Holders_and_Fuses:Fuse_TE5_Littlefuse-395Series" H 1800 4250 50  0001 L CNN
+F 3 "~" H 1750 4450 50  0001 C CNN
+	1    1750 4450
+	0    1    1    0
+$EndComp
+Wire Wire Line
+	1900 4450 2050 4450
+Wire Wire Line
+	1150 4450 1600 4450
+$Comp
+L diode:1N4004 D2
+U 1 1 5EE17EBE
+P 1050 5750
+F 0 "D2" V 1004 5829 50  0000 L CNN
+F 1 "1N4004" V 1095 5829 50  0000 L CNN
+F 2 "Diodes_THT:D_DO-41_SOD81_P10.16mm_Horizontal" H 1050 5575 50  0001 C CNN
+F 3 "http://www.vishay.com/docs/88503/1n4001.pdf" H 1050 5750 50  0001 C CNN
+	1    1050 5750
+	0    1    1    0
+$EndComp
+Wire Wire Line
+	1050 5600 1050 5450
+Wire Wire Line
+	1050 6050 1050 5900
+$Comp
+L power:+BATT #PWR?
+U 1 1 5EE1FB8D
+P 2050 4450
+AR Path="/5EE1FB8D" Ref="#PWR?"  Part="1"
+AR Path="/5EDE387A/5EE1FB8D" Ref="#PWR0123"  Part="1"
+F 0 "#PWR0123" H 2050 4300 50  0001 C CNN
+F 1 "+BATT" H 2065 4623 50  0000 C CNN
+F 2 "" H 2050 4450 50  0001 C CNN
+F 3 "" H 2050 4450 50  0001 C CNN
+	1    2050 4450
+	1    0    0    -1
+$EndComp
+$Comp
+L power:-BATT #PWR?
+U 1 1 5EE1FEB1
+P 1550 4550
+AR Path="/5EE1FEB1" Ref="#PWR?"  Part="1"
+AR Path="/5EDE387A/5EE1FEB1" Ref="#PWR0124"  Part="1"
+F 0 "#PWR0124" H 1550 4400 50  0001 C CNN
+F 1 "-BATT" V 1550 4700 50  0000 L CNN
+F 2 "" H 1550 4550 50  0001 C CNN
+F 3 "" H 1550 4550 50  0001 C CNN
+	1    1550 4550
+	0    1    1    0
+$EndComp
+Wire Notes Line
+	650  4950 2850 4950
+Wire Notes Line
+	2850 4950 2850 6450
+Wire Notes Line
+	2850 6450 650  6450
+Wire Notes Line
+	650  6450 650  4950
+Text Notes 700  5150 0    118  ~ 0
+Verpolschutz Battery
 $EndSCHEMATC

Commit message: Backup Pins added (6 IOs Vcc GND)
Parts:
- added J11: Conn_01x02_Male, Pin_Headers:Pin_Header_Straight_1x02_Pitch2.54mm_SMD_Pin1Left, symbol conn:Conn_01x02_Male
- D2: footprint Diodes_THT:D_DO-41_SOD81_P10.16mm_Horizontal -> Diodes_THT:D_DO-41_SOD81_P5.08mm_Vertical_KathodeUp
Connections:
- wire segments 22 -> 26
Changed lines of the file:
@@
 F 0 "D2" V 1004 5829 50  0000 L CNN
 F 1 "1N4004" V 1095 5829 50  0000 L CNN
-F 2 "Diodes_THT:D_DO-41_SOD81_P10.16mm_Horizontal" H 1050 5575 50  0001 C CNN
+F 2 "Diodes_THT:D_DO-41_SOD81_P5.08mm_Vertical_KathodeUp" H 1050 5575 50  0001 C CNN
 F 3 "http://www.vishay.com/docs/88503/1n4001.pdf" H 1050 5750 50  0001 C CNN
 	1    1050 5750
@@
 Text Notes 700  5150 0    118  ~ 0
 Verpolschutz Battery
+$Comp
+L conn:Conn_01x02_Male J?
+U 1 1 5EED3385
+P 3000 1550
+AR Path="/5EED3385" Ref="J?"  Part="1"
+AR Path="/5EDE387A/5EED3385" Ref="J11"  Part="1"
+F 0 "J11" H 3108 1731 50  0000 C CNN
+F 1 "Conn_01x02_Male" H 3108 1640 50  0000 C CNN
+F 2 "Pin_Headers:Pin_Header_Straight_1x02_Pitch2.54mm_SMD_Pin1Left" H 3000 1550 50  0001 C CNN
+F 3 "~" H 3000 1550 50  0001 C CNN
+F 4 "Batterie Connector (bevorzugt Reichelt da direkt als Kabelset!)" H 3000 1550 50  0001 C CNN "Bemerkung"
+F 5 "https://www.conrad.de/de/p/bkl-electronic-stiftleiste-standard-anzahl-reihen-1-polzahl-je-reihe-40-10120513-1-393494.html" H 3000 1550 50  0001 C CNN "Conrad"
+F 6 "https://www.reichelt.de/platinensteckverbinder-gerade-weiss-2-polig-ps-25-2g-ws-p14825.html" H 3000 1550 50  0001 C CNN "Reichelt"
+F 7 "https://www.segor.de/#Q=SL1x40-180G%252F13%252C8&M=1" H 3000 1550 50  0001 C CNN "Segor.de"
+	1    3000 1550
+	1    0    0    -1
+$EndComp
+$Comp
+L power:+3.3V #PWR?
+U 1 1 5EED3AE0
+P 3500 1500
+AR Path="/5EED3AE0" Ref="#PWR?"  Part="1"
+AR Path="/5EDE387A/5EED3AE0" Ref="#PWR04"  Part="1"
+F 0 "#PWR04" H 3500 1350 50  0001 C CNN
+F 1 "+3.3V" H 3515 1673 50  0000 C CNN
+F 2 "" H 3500 1500 50  0001 C CNN
+F 3 "" H 3500 1500 50  0001 C CNN
+	1    3500 1500
+	1    0    0    -1
+$EndComp
+$Comp
+L power:GND #PWR?
+U 1 1 5EED3F0D
+P 3500 1700
+AR Path="/5EED3F0D" Ref="#PWR?"  Part="1"
+AR Path="/5EDE387A/5EED3F0D" Ref="#PWR05"  Part="1"
+F 0 "#PWR05" H 3500 1450 50  0001 C CNN
+F 1 "GND" H 3505 1527 50  0000 C CNN
+F 2 "" H 3500 1700 50  0001 C CNN
+F 3 "" H 3500 1700 50  0001 C CNN
+	1    3500 1700
+	1    0    0    -1
+$EndComp
+Wire Wire Line
+	3200 1550 3500 1550
+Wire Wire Line
+	3500 1550 3500 1500
+Wire Wire Line
+	3200 1650 3500 1650
+Wire Wire Line
+	3500 1650 3500 1700
 $EndSCHEMATC

Commit message: updated D2 to DO-201 package
Parts:
- D2: value 1N4004 -> SB560; footprint Diodes_THT:D_DO-41_SOD81_P5.08mm_Vertical_KathodeUp -> Diode_THT:D_DO-201AE_P12.70mm_Horizontal; symbol diode:1N4004 -> diode:1N5820
Changed lines of the file:
@@
 EESchema Schematic File Version 4
+LIBS:OpenBikeSensor_pcb_flippedPower_b-cache
 EELAYER 30 0
 EELAYER END
@@
 	1150 4450 1600 4450
 $Comp
-L diode:1N4004 D2
+L diode:1N5820 D2
 U 1 1 5EE17EBE
 P 1050 5750
 F 0 "D2" V 1004 5829 50  0000 L CNN
-F 1 "1N4004" V 1095 5829 50  0000 L CNN
-F 2 "Diodes_THT:D_DO-41_SOD81_P5.08mm_Vertical_KathodeUp" H 1050 5575 50  0001 C CNN
+F 1 "SB560" V 1095 5829 50  0000 L CNN
+F 2 "Diode_THT:D_DO-201AE_P12.70mm_Horizontal" H 1050 5575 50  0001 C CNN
 F 3 "http://www.vishay.com/docs/88503/1n4001.pdf" H 1050 5750 50  0001 C CNN
 	1    1050 5750

Commit message: clean up model references and add missing libraries
Parts:
- D2: symbol diode:1N5820 -> Diode:1N5820
- F1: symbol device:Polyfuse -> Device:Polyfuse
- J1, J6: footprint Pin_Headers:Pin_Header_Straight_1x02_Pitch2.54mm -> Connector_PinHeader_2.54mm:PinHeader_1x02_P2.54mm_Vertical; symbol conn:Conn_01x02_Male -> Connector:Conn_01x02_Male
- J11: symbol conn:Conn_01x02_Male -> Connector:Conn_01x02_Male
- U2: footprint (none) -> Custom_Modules:LM2596_Mini
Changed lines of the file:
@@
 EESchema Schematic File Version 4
-LIBS:OpenBikeSensor_pcb_flippedPower_b-cache
 EELAYER 30 0
 EELAYER END
@@
 F 0 "U2" H 8525 2765 50  0000 C CNN
 F 1 "LM2596_mini" H 8525 2674 50  0000 C CNN
-F 2 "" H 8500 2650 50  0001 C CNN
+F 2 "Custom_Modules:LM2596_Mini" H 8500 2650 50  0001 C CNN
 F 3 "" H 8500 2650 50  0001 C CNN
 F 4 "obsolet" H 8550 2300 50  0001 C CNN "Optional"
@@
 	2250 3700 2400 3700
 $Comp
-L conn:Conn_01x02_Male J?
+L Connector:Conn_01x02_Male J?
 U 1 1 5EDFEA52
 P 2650 3100
@@
 F 0 "J6" V 2450 3050 50  0000 C CNN
 F 1 "Conn_01x02_Male" V 2550 3100 50  0000 C CNN
-F 2 "Pin_Headers:Pin_Header_Straight_1x02_Pitch2.54mm" H 2650 3100 50  0001 C CNN
+F 2 "Connector_PinHeader_2.54mm:PinHeader_1x02_P2.54mm_Vertical" H 2650 3100 50  0001 C CNN
 F 3 "~" H 2650 3100 50  0001 C CNN
 F 4 "Switch Connector" H 2650 3100 50  0001 C CNN "Bemerkung"
@@
 $EndComp
 $Comp
-L conn:Conn_01x02_Male J?
+L Connector:Conn_01x02_Male J?
 U 1 1 5EE082AD
 P 950 4450
@@
 F 0 "J1" H 1058 4631 50  0000 C CNN
 F 1 "Conn_01x02_Male" H 1058 4540 50  0000 C CNN
-F 2 "Pin_Headers:Pin_Header_Straight_1x02_Pitch2.54mm" H 950 4450 50  0001 C CNN
+F 2 "Connector_PinHeader_2.54mm:PinHeader_1x02_P2.54mm_Vertical" H 950 4450 50  0001 C CNN
 F 3 "~" H 950 4450 50  0001 C CNN
 F 4 "Batterie Connector (bevorzugt Reichelt da direkt als Kabelset!)" H 950 4450 50  0001 C CNN "Bemerkung"
@@
 $EndComp
 $Comp
-L device:Polyfuse F1
+L Device:Polyfuse F1
 U 1 1 5EE15FB8
 P 1750 4450
@@
 	1150 4450 1600 4450
 $Comp
-L diode:1N5820 D2
+L Diode:1N5820 D2
 U 1 1 5EE17EBE
 P 1050 5750
@@
 Verpolschutz Battery
 $Comp
-L conn:Conn_01x02_Male J?
+L Connector:Conn_01x02_Male J?
 U 1 1 5EED3385
 P 3000 1550
